Commit message: Abb fixups

File: godel_robot_config/urdf/irb2400_workspace.xacro (robot description, xacro)
@@ -3,5 +3,5 @@
   <xacro:include filename="$(find abb_irb2400_support)/urdf/irb2400_macro.xacro"/>
   <xacro:include filename="$(find godel_robot_config)/urdf/workspace_components.xacro"/>
-  <xacro:include filename="$(find godel_robot_config)/urdf/blending_eff_macro.xacro"/>
+  <xacro:include filename="$(find godel_robot_config)/urdf/abb_blending_eff_macro.xacro"/>
   <!-- property list -->
   <xacro:property name="workcell_height" value="1"/>
@@ -19,5 +19,5 @@
     <parent link="tool0"/>
     <child link="eff_frame"/>
-    <origin xyz="0 ${coupler_height} 0" rpy="0.0 0.0 3.1416"/>
+    <origin xyz="0 ${coupler_height} 0" rpy="0.0 0.0 0.0"/>
   </joint>
   <!-- start of arm-workcell joint definitions -->
