Commit message: The number of changes is getting out of control

File: godel_robot_config/urdf/abb_blending_eff_macro.xacro (robot description, xacro)
@@ -23,10 +23,8 @@
 			</visual>
 			<collision>
+				<origin xyz="0 0 0.1"/>
 				<geometry>
-					<mesh filename="package://godel_robot_config/meshes/SWRI_Tool_cf.stl" />
-				</geometry>
-				<material name="another_blue2">
-					<color rgba="0.38 0.54 0.83 1"/>
-				</material>
+          <box size="0.25 0.065 0.04"/>
+        </geometry>
 			</collision>
 		</link>

File: godel_robot_config/urdf/blending_eff_macro.xacro (robot description, xacro)
@@ -32,5 +32,5 @@
 		<link name="${prefix}keyence_mount"/>
 		<xacro:kinect2_sensor_definitions prefix="${prefix}" parent_link="${prefix}kinect2_mount"
-				x_val="0.01468947476802748" y_val="-0.06367377711162475" z_val="-0.01960868079016488" roll="-0.008749106789621127" pitch="-0.03236299096413636" yaw="0.01705034660528017"/>
+				x_val="0.01434829753039301" y_val="-0.06323676415307219" z_val="-0.01938774892474541" roll="-0.01029402937163579" pitch="-0.02742921475882609" yaw="0.01025802202749901"/>
 		<!-- Keyence sensor -->
 		<xacro:keyence_lj_v7080 prefix="${prefix}keyence_" />

File: godel_robot_config/urdf/kinect2_sensor_macro.xacro (robot description, xacro)
@@ -13,5 +13,5 @@
     <!-- sensor links -->
     <link name="${prefix}kinect2_frame">
-      <visual>
+      <!-- <visual>
         <origin rpy="0 0 0" xyz="0 0 0"/>
         <geometry>
@@ -25,5 +25,5 @@
           <box size="${asus_width} ${asus_length} ${asus_height}"/>
         </geometry>
-      </collision>
+      </collision> -->
     </link>
     <link name="${prefix}kinect2_ir_frame">

File: keyence_ljv_description/urdf/lj_v7080_macro.xacro (robot description, xacro)
@@ -8,5 +8,5 @@
   <xacro:macro name="keyence_lj_v7080" params="prefix">
     <link name="${prefix}base_link">
-      <visual>
+     <!--  <visual>
         <origin xyz="${box_l/-2} 0 0" rpy="0 0 0"/>
         <geometry>
@@ -22,5 +22,5 @@
           <box size="${box_l} ${box_w} ${box_h}"/>
         </geometry>
-      </collision>
+      </collision> -->
     </link>
     <link name="${prefix}sensor_aperture_frame" />

Commit message: Updated the abb eef macro to match the fancy new models

File: godel_robot_config/urdf/abb_blending_eff_macro.xacro (robot description, xacro)
@@ -4,41 +4,53 @@
 	<xacro:include filename="$(find keyence_ljv_description)/urdf/lj_v7080_macro.xacro"/>
 	<!-- parameter list -->
-	<xacro:property name="gripper_length" value="0.218"/>
-	<xacro:property name="gripper_width" value="0.0"/>
-	<xacro:property name="gripper_height" value="0.0"/>
-	<xacro:property name="TCP_X" value="-0.175286"/>
-	<xacro:property name="TCP_Y" value="-0.088502"/>
-	<xacro:property name="TCP_Z" value="0.056356"/>
+	<xacro:property name="blend_tcp_x" value="-0.175286"/>
+	<xacro:property name="blend_tcp_y" value="-0.088502"/>
+	<xacro:property name="blend_tcp_z" value="0.056356"/>
+	<xacro:property name="keyence_optical_x" value="0.3016"/>
+	<xacro:property name="keyence_optical_y" value="-0.057"/>
+	<xacro:property name="keyence_optical_z" value="0.088502"/>
+	<xacro:property name="kinect_optical_x" value="0.09"/>
+	<xacro:property name="kinect_optical_y" value="-0.065"/>
+	<xacro:property name="kinect_optical_z" value="0.15"/>
 	<xacro:macro name="blending_eff_definition" params="prefix eff_adjustment">
-			<!-- link definition -->
+		<!-- Link Interface -->
+		<!-- Base link - attach your robot to this link -->
 		<link name="${prefix}eff_frame"/>
+		<!-- Blend tool tip link -->
+		<link name="${prefix}tcp_frame"/>
+		<!-- Camera movement target frame  -->
+		<!-- Keyence laser scanner target frame -->
+		<link name="${prefix}keyence_tcp_frame" />
+		<!-- Intermediate Links -->
 		<link name="${prefix}gripper_body">
 			<visual>
 				<geometry>
-					<mesh filename="package://godel_robot_config/meshes/SWRI_Tool_cf.stl" />
+					<mesh filename="package://godel_robot_config/meshes/visual/blending_eff.stl" />
 				</geometry>
-				<material name="silver">
-					<color rgba="0.8 0.8 0.8 1"/>
+				<material name="grey">
+					<color rgba="0.5 0.5 0.5 1.0"/>
 				</material>
 			</visual>
 			<collision>
-				<origin xyz="0 0 0.1"/>
 				<geometry>
-          <box size="0.25 0.065 0.04"/>
+          <!-- <mesh filename="package://godel_robot_config/meshes/visual/blending_eff.stl" /> -->
+          <cylinder length="0.01" radius="0.01"/>
         </geometry>
 			</collision>
 		</link>
-		<link name="${prefix}tcp_frame"/>
 		<link name="${prefix}kinect2_mount"/>
-		<link name="${prefix}keyence_mount"/>
 		<xacro:kinect2_sensor_definitions prefix="${prefix}" parent_link="${prefix}kinect2_mount"
 				x_val="0.01468947476802748" y_val="-0.06367377711162475" z_val="-0.01960868079016488" roll="-0.008749106789621127" pitch="-0.03236299096413636" yaw="0.01705034660528017"/>
 		<!-- Keyence sensor -->
-		<xacro:keyence_lj_v7080 prefix="${prefix}keyence_" />
-		<link name="${prefix}keyence_tcp_frame" />
-		<joint name="${prefix}keyence_to_keyence_tcp_frame" type="fixed">
+		<link name="${prefix}keyence_sensor_optical_frame"/>
+		<joint name="${prefix}gripper_to_keyence_optical" type="fixed">
+			<parent link="${prefix}gripper_body"/>
+			<child link="${prefix}keyence_sensor_optical_frame"/>
+			<origin xyz="${keyence_optical_x} ${keyence_optical_y} ${keyence_optical_z}" rpy="0 1.5705 3.14159"/>
+		</joint>
+		<joint name="${prefix}keyence_optical_to_keyence_tcp" type="fixed">
 			<parent link="${prefix}keyence_sensor_optical_frame"/>
 			<child link="${prefix}keyence_tcp_frame"/>
-			<origin xyz="0.05 0 0" rpy="0 3.14159 0"/>
+			<origin rpy="0 3.14159 0"/>
 		</joint>
 		<!-- joint definitions -->
@@ -46,25 +58,14 @@
 			<parent link="${prefix}eff_frame"/>
 			<child link="${prefix}gripper_body"/>
-			<origin xyz="0 0 ${gripper_height * 0.5}" rpy="0 0 0"/>
 		</joint>
-		<joint name="${prefix}eff_frame_to_kinect2_mount" type="fixed">
-			<parent link="${prefix}eff_frame"/>
+		<joint name="${prefix}gripper_to_kinect2_mount" type="fixed">
+			<parent link="${prefix}gripper_body"/>
 			<child link="${prefix}kinect2_mount"/>
-			<origin xyz="0 0 0.150" rpy="3.14 0 ${2.09+3.141592653589793}"/>
+			<origin xyz="${kinect_optical_x} ${kinect_optical_y} ${kinect_optical_z}" rpy="0 3.14159 -1.5705"/>
 		</joint>
 		<joint name="${prefix}gripper_to_tcp" type="fixed">
 			<parent link="${prefix}gripper_body"/>
 			<child link="${prefix}tcp_frame"/>
-			<origin xyz="${TCP_X} ${TCP_Y} ${TCP_Z}" rpy="0 -1.570796326 0"/>
-		</joint>
-		<joint name="${prefix}gripper_to_keyence_mount" type="fixed">
-			<parent link="${prefix}gripper_body" />
-			<child link="${prefix}keyence_mount"/>
-			<origin xyz="-0.16 0 0.08" rpy="0 1.570796326 0" />
-		</joint>
-		<joint name="${prefix}keyence_mount_to_keyence" type="fixed">
-			<parent link="${prefix}keyence_mount"/>
-			<child link="${prefix}keyence_base_link"/>
-			<origin xyz="0 0 0" rpy="0 0 1.570796326"/>
+			<origin xyz="${blend_tcp_x} ${blend_tcp_y} ${blend_tcp_z}" rpy="0 -1.570796326 0"/>
 		</joint>
 	</xacro:macro>

File: godel_robot_config/urdf/irb2400_workspace.xacro (robot description, xacro)
@@ -6,7 +6,6 @@
   <!-- property list -->
   <xacro:property name="workcell_height" value="1"/>
-  <xacro:property name="coupler_height" value="0.0"/> <!--"0.087"-->
   <xacro:property name="arm_prefix" value=""/>
-  <xacro:property name="no_go_height" value="0.1"/>
+  <xacro:property name="no_go_height" value="0.01"/>
   <!-- instantiating workcell definitions -->
   <xacro:workcell_zone1_components/>
@@ -19,5 +18,4 @@
     <parent link="tool0"/>
     <child link="eff_frame"/>
-    <origin xyz="0 ${coupler_height} 0" rpy="0.0 0.0 0.0"/>
   </joint>
   <!-- start of arm-workcell joint definitions -->

Commit message: Robot description updates

File: godel_robot_config/urdf/abb_blending_eff_macro.xacro (robot description, xacro)
@@ -4,5 +4,5 @@
 	<xacro:include filename="$(find keyence_ljv_description)/urdf/lj_v7080_macro.xacro"/>
 	<!-- parameter list -->
-	<xacro:property name="blend_tcp_x" value="-0.175286"/>
+	<xacro:property name="blend_tcp_x" value="-0.180286"/>
 	<xacro:property name="blend_tcp_y" value="-0.088502"/>
 	<xacro:property name="blend_tcp_z" value="0.056356"/>
@@ -33,7 +33,8 @@
 			</visual>
 			<collision>
+				<origin xyz="0 0 0.05"/>
 				<geometry>
-          <!-- <mesh filename="package://godel_robot_config/meshes/visual/blending_eff.stl" /> -->
-          <cylinder length="0.01" radius="0.01"/>
+          <!-- <mesh filename="package://godel_robot_config/meshes/collision/blending_eff.stl" /> -->
+          <cylinder length="0.02" radius="0.01"/>
         </geometry>
 			</collision>
@@ -41,5 +42,5 @@
 		<link name="${prefix}kinect2_mount"/>
 		<xacro:kinect2_sensor_definitions prefix="${prefix}" parent_link="${prefix}kinect2_mount"
-				x_val="0.01468947476802748" y_val="-0.06367377711162475" z_val="-0.01960868079016488" roll="-0.008749106789621127" pitch="-0.03236299096413636" yaw="0.01705034660528017"/>
+				x_val="0.02900174412393907" y_val="0.04095818230741284" z_val="-0.01883104837032643" roll="-0.01098684541346244" pitch="0.03293993758199074" yaw="0.008473303411297784"/>
 		<!-- Keyence sensor -->
 		<link name="${prefix}keyence_sensor_optical_frame"/>
@@ -47,5 +48,5 @@
 			<parent link="${prefix}gripper_body"/>
 			<child link="${prefix}keyence_sensor_optical_frame"/>
-			<origin xyz="${keyence_optical_x} ${keyence_optical_y} ${keyence_optical_z}" rpy="0 1.5705 3.14159"/>
+			<origin xyz="${keyence_optical_x} ${keyence_optical_y} ${keyence_optical_z}" rpy="0 1.5707963267948966 3.141592653589793"/>
 		</joint>
 		<joint name="${prefix}keyence_optical_to_keyence_tcp" type="fixed">
@@ -62,5 +63,5 @@
 			<parent link="${prefix}gripper_body"/>
 			<child link="${prefix}kinect2_mount"/>
-			<origin xyz="${kinect_optical_x} ${kinect_optical_y} ${kinect_optical_z}" rpy="0 3.14159 -1.5705"/>
+			<origin xyz="${kinect_optical_x} ${kinect_optical_y} ${kinect_optical_z}" rpy="0 3.141592653589793 1.5707963267948966"/>
 		</joint>
 		<joint name="${prefix}gripper_to_tcp" type="fixed">

File: godel_robot_config/urdf/blending_eff_macro.xacro (robot description, xacro)
@@ -32,12 +32,12 @@
 		<link name="${prefix}keyence_mount"/>
 		<xacro:kinect2_sensor_definitions prefix="${prefix}" parent_link="${prefix}kinect2_mount"
-				x_val="0.01434829753039301" y_val="-0.06323676415307219" z_val="-0.01938774892474541" roll="-0.01029402937163579" pitch="-0.02742921475882609" yaw="0.01025802202749901"/>
+				x_val="0.01342977865645872" y_val="-0.05686282224354644" z_val="-0.01969773723914273" roll="0.01321096089091111" pitch="-0.0264784868525508" yaw="-0.008407104830530813"/>
 		<!-- Keyence sensor -->
 		<xacro:keyence_lj_v7080 prefix="${prefix}keyence_" />
 		<link name="${prefix}keyence_tcp_frame" />
 		<joint name="${prefix}keyence_to_keyence_tcp_frame" type="fixed">
-			<parent link="${prefix}keyence_sensor_optical_frame"/>
+			<parent link="${prefix}gripper_body"/>
 			<child link="${prefix}keyence_tcp_frame"/>
-			<origin xyz="0.05 0 0" rpy="0 3.14159 0"/>
+			<origin xyz="-0.3016 0.028 0.0935" rpy="0 1.57 3.14159"/>
 		</joint>
 		<!-- joint definitions -->
@@ -55,5 +55,5 @@
 			<parent link="${prefix}gripper_body"/>
 			<child link="${prefix}tcp_frame"/>
-			<origin xyz="${gripper_length} 0 ${eff_adjustment}" rpy="0 1.570796326 0"/>
+			<origin xyz="0.2 0 0.05636" rpy="0 1.570796326 0"/>
 		</joint>
 		<joint name="${prefix}gripper_to_keyence_mount" type="fixed">

File: godel_robot_config/urdf/irb6640_workspace.xacro (robot description, xacro)
@@ -3,5 +3,5 @@
   <xacro:include filename="$(find abb_irb6600_support)/urdf/irb6640_macro.xacro"/>
   <xacro:include filename="$(find godel_robot_config)/urdf/workspace_components.xacro"/>
-  <xacro:include filename="$(find godel_robot_config)/urdf/blending_eff_macro.xacro"/>
+  <xacro:include filename="$(find godel_robot_config)/urdf/abb_blending_eff_macro.xacro"/>
   <!-- property list -->
   <xacro:property name="workcell_height" value="1"/>
@@ -19,5 +19,5 @@
     <parent link="tool0"/>
     <child link="eff_frame"/>
-    <origin xyz="0 ${coupler_height} 0" rpy="0.0 0.0 3.1416"/>
+    <origin xyz="0 ${coupler_height} 0" rpy="0.0 0.0 0.0"/>
   </joint>
   <!-- start of arm-workcell joint definitions -->

File: godel_robot_config/urdf/workspace_components_swri.xacro (robot description, xacro)
@@ -3,6 +3,6 @@
 	<!-- property list -->
 	<xacro:property name="workcell_height" value="1"/>
-	<xacro:property name="workcell_length" value="2.775"/>
-	<xacro:property name="workcell_width" value="2.220"/>
+	<xacro:property name="workcell_length" value="2.775"/> <!--2.775 -->
+ 	<xacro:property name="workcell_width" value="2.220"/>
 	<xacro:property name="workcell_thickness" value="0.04"/>
 	<!-- color macros -->
@@ -102,9 +102,9 @@
 		</joint>
 		<xacro:workcell_element name="front_wall1" parent="world_frame"
-			 length="0.1" width="2.220" height="${workcell_height}" offset_x="1.3375" offset_y="0"/>
+			 length="0.1" width="2.220" height="${workcell_height}" offset_x="1.29" offset_y="0"/> <!-- 1.3375 -->
 		<xacro:workcell_element name="back_wall1" parent="world_frame"
 			 length="0.04" width="2.00" height="${workcell_height}" offset_x="0.02" offset_y="0"/>
 		<xacro:workcell_element name="left_wall1" parent="world_frame"
-			 length="1.221" width="0.1" height="${workcell_height}" offset_x="0.687" offset_y="1.060"/>
+			 length="1.221" width="0.1" height="${workcell_height}" offset_x="0.687" offset_y="0.9"/> <!--1.060-->
 		<xacro:workcell_element name="right_wall1" parent="world_frame"
 			 length="1.221" width="0.1" height="${workcell_height}" offset_x="0.687" offset_y="-1.060"/>

Commit message: Updated 2600 workspace and related settings (including camera cal)

File: godel_robot_config/urdf/abb_blending_eff_macro.xacro (robot description, xacro)
@@ -4,5 +4,6 @@
 	<xacro:include filename="$(find keyence_ljv_description)/urdf/lj_v7080_macro.xacro"/>
 	<!-- parameter list -->
-	<xacro:property name="blend_tcp_x" value="-0.180286"/>
+	<!-- -0.18415 -->
+	<xacro:property name="blend_tcp_x" value="-0.18415"/>
 	<xacro:property name="blend_tcp_y" value="-0.088502"/>
 	<xacro:property name="blend_tcp_z" value="0.056356"/>
@@ -33,5 +34,5 @@
 			</visual>
 			<collision>
-				<origin xyz="0 0 0.05"/>
+				<origin xyz="0 0 300.0"/>
 				<geometry>
           <!-- <mesh filename="package://godel_robot_config/meshes/collision/blending_eff.stl" /> -->
@@ -42,5 +43,5 @@
 		<link name="${prefix}kinect2_mount"/>
 		<xacro:kinect2_sensor_definitions prefix="${prefix}" parent_link="${prefix}kinect2_mount"
-				x_val="0.02900174412393907" y_val="0.04095818230741284" z_val="-0.01883104837032643" roll="-0.01098684541346244" pitch="0.03293993758199074" yaw="0.008473303411297784"/>
+				x_val="0.04820261546730869" y_val="-0.01114874709948466" z_val="-0.02950381228410577" roll="0.007508267029451446" pitch="-0.02318953773117859" yaw="-0.01522249965961855"/>
 		<!-- Keyence sensor -->
 		<link name="${prefix}keyence_sensor_optical_frame"/>
@@ -63,5 +64,5 @@
 			<parent link="${prefix}gripper_body"/>
 			<child link="${prefix}kinect2_mount"/>
-			<origin xyz="${kinect_optical_x} ${kinect_optical_y} ${kinect_optical_z}" rpy="0 3.141592653589793 1.5707963267948966"/>
+			<origin xyz="${kinect_optical_x} ${kinect_optical_y} ${kinect_optical_z}" rpy="0 3.141592653589793 -1.5707963267948966"/>
 		</joint>
 		<joint name="${prefix}gripper_to_tcp" type="fixed">

File: godel_robot_config/urdf/irb2600_workspace.xacro (robot description, xacro)
@@ -10,5 +10,5 @@
   <xacro:property name="no_go_height" value="0.1"/>
   <!-- instantiating workcell definitions -->
-  <xacro:workcell_zone1_components/>
+  <!-- <xacro:workcell_zone1_components/> -->
   <!-- instantiating arm  -->
   <xacro:abb_irb2600 prefix="${arm_prefix}"/>
@@ -31,9 +31,4 @@
      from getting too close to the table. Descartes is still unawares, though -->
   <link name="no_go_zone">
-    <collision>
-      <geometry>
-        <box size="0.8 2.220 ${no_go_height}"/>
-      </geometry>
-    </collision>
   </link>
   <joint name="world_to_no_go" type="fixed">
