Commit message: Huge changes to the calibration portion. New files for each of the supported robots.

File: godel_calibration_config/urdf/calib_kinect2_sensor_macro.xacro (robot description, xacro)
@@ -16,11 +16,11 @@
     <!-- sensor links -->
     <link name="${prefix}kinect2_frame">
-      <visual>
-        <origin rpy="0 0 0" xyz="0 0 0"/>
+      <!-- <visual> -->
+       <!--  <origin rpy="0 0 0" xyz="0 0 0"/>
         <geometry>
           <box size="${asus_width} ${asus_length} ${asus_height}"/>
         </geometry>
         <material name="${prefix}dark_silver"/>
-      </visual>
+      </visual> -->
       <!-- <collision>
         <origin rpy="0 0 0" xyz="0 0 0"/>
