Commit message: Temporarily removed the collision model from the keyence itself. Instead it's being incorporated as part of a larger mesh

File: keyence_ljv_description/urdf/lj_v7080_macro.xacro (robot description, xacro)
@@ -8,5 +8,5 @@
   <xacro:macro name="keyence_lj_v7080" params="prefix">
     <link name="${prefix}base_link">
-     <!--  <visual>
+      <!-- <visual>
         <origin xyz="${box_l/-2} 0 0" rpy="0 0 0"/>
         <geometry>
