Commit message: Updated the 2400's URDF and launch files to work as they should

File: godel_robots/abb/godel_irb2400/godel_irb2400_support/urdf/abb_blending_eff_macro.xacro (robot description, xacro)
@@ -43,10 +43,10 @@
     <xacro:unless value="${calibration}">
       <xacro:kinect2_sensor_definitions prefix="${prefix}" parent_link="${prefix}kinect2_mount"
-        x_val="0.04034282619366366"
-        y_val="-0.01220757033046958"
-        z_val="-0.02365034085440264"
-        roll="0.001680561166170003"
-        pitch="0.01944455166614176"
-        yaw="-0.02261820677639799"/>
+        x_val="-0.057131"
+        y_val="-0.109731"
+        z_val="-0.016649"
+        roll="1.594112"
+        pitch="0.012460"
+        yaw="-1.572763"/>
     </xacro:unless>
     <joint name="${prefix}gripper_to_keyence_optical" type="fixed">
@@ -74,4 +74,10 @@
       <origin xyz="${blend_tcp_x} ${blend_tcp_y} ${blend_tcp_z}" rpy="0 -1.5707963267948966 0"/>
     </joint>
+    <link name="${prefix}kinect2_move_frame" />
+    <joint name="${prefix}kinect2_move_frame_joint" type="fixed">
+      <parent link="${prefix}kinect2_mount"/>
+      <child link="${prefix}kinect2_move_frame"/>
+      <origin rpy="3.14159 0 3.14159" xyz="0 0 0"/>
+    </joint>
   </xacro:macro>
 </robot>

File: godel_robots/godel_robot_resources/urdf/calib_kinect2_sensor_macro.xacro (robot description, xacro)
@@ -4,10 +4,4 @@
   <xacro:macro name="calib_kinect2_sensor_definitions" params="prefix parent_link">
     <link name="${prefix}kinect2_link"/>
-    <link name="${prefix}kinect2_move_frame" />
-    <joint name="${prefix}kinect2_move_frame_joint" type="fixed">
-      <parent link="${prefix}kinect2_link"/>
-      <child link="${prefix}kinect2_move_frame"/>
-      <origin rpy="0 0 0" xyz="0 0 0"/>
-    </joint>
     <xacro:calibration_definitions child_link="${prefix}kinect2_link" parent_link="${parent_link}" />
   </xacro:macro>

File: godel_robots/godel_robot_resources/urdf/kinect2_sensor_macro.xacro (robot description, xacro)
@@ -3,10 +3,4 @@
   <xacro:macro name="kinect2_sensor_definitions" params="prefix parent_link x_val y_val z_val roll pitch yaw">
     <link name="${prefix}kinect2_link"/>
-    <link name="${prefix}kinect2_move_frame" />
-    <joint name="${prefix}kinect2_move_frame_joint" type="fixed">
-      <parent link="${prefix}kinect2_link"/>
-      <child link="${prefix}kinect2_move_frame"/>
-      <origin rpy="0 0 0" xyz="0 0 0"/>
-    </joint>
     <joint name="${parent_link}_to_kinect2_link" type="fixed">
       <parent link="${parent_link}"/>
